File: Hardware/sus_gimbal_controller/untitled.kicad_sch (KiCad schematic)
At the start: 103 parts, among them J1 8P8C_LED_Shielded, Q1 NMOS, Q10 NMOS, Q11 NMOS, Q12 NMOS, Q13 NMOS, Q14 NMOS, Q15 NMOS, Q16 NMOS, Q17 NMOS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

Commit message: Added datasheet
real
Parts:
- U4: footprint (none) -> QFN
Changed lines of the file:
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@@
 	)
 	(symbol
+		(lib_name "MRDT_Devices:DRV8239")
 		(lib_id "MRDT_Devices:DRV8239")
 		(at 377.19 121.92 0)
@@
 			)
 		)
-		(property "Footprint" ""
+		(property "Footprint" "QFN"
 			(at 355.6 160.02 0)
 			(effects
@@
 			)
 		)
-		(property "Datasheet" ""
+		(property "Datasheet" "https://www.ti.com/lit/ds/symlink/drv8329.pdf?ts=1731490781953&ref_url=https%253A%252F%252Fwww.ti.com%252Fproduct%252FDRV8329%253FkeyMatch%253DDRV8329A%2526tisearch%253Duniversal_search%2526usecase%253Dpartmatches"
 			(at 355.6 160.02 0)
 			(effects

Commit message: filepath
to be fixed
Parts:
- C13: value 0.1uf -> 1uf
- C9: value 470 uF -> 470 nF
Connections:
- net CS: no longer Q10.3 (S), Q12.3 (S), Q14.3 (S), Q16.3 (S), Q18.3 (S), Q4.3 (S), Q8.3 (S)
- net GHA: now also R5.1
- net GHB: no longer R5.1
- net GLA: now also R6.1
- net GLB: no longer R6.1
- net GND: now also U4.25 (AGND)
- net SO (1): no longer U7.2 (SO)
- net SO (3): now also U7.2 (SO)
- new net CS_1: Q12.3 (S), Q4.3 (S), Q8.3 (S)
- new net CS_2: Q10.3 (S), Q18.3 (S)
- new net CS_3: Q14.3 (S), Q16.3 (S)
- no-connect marks 30 -> 31
Other:
- moved on the sheet: C10
