File: Hardware/BrushlessGimbalController_Hardware/BrushlessGimbalController_Hardware.kicad_pcb (KiCad board)
At the start: 2 copper layers, 305.1 x 210.8 mm, 126 parts, among them J1 8P8C_LED_Shielded, Q1 NMOS, Q10 NMOS, Q11 NMOS, Q12 NMOS, Q13 NMOS, Q14 NMOS, Q15 NMOS, Q16 NMOS, Q17 NMOS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

Commit message: Layout revisions
Layout revisions implemented from conversation with Drew
Edge cuts added
Vias added to ground planes
Ethernet connector moved to not attach to Teensey
Hopefully ready for order whenever next board order date is
Parts:
- added REF**: MountingHole_3mm, MountingHole:MountingHole_3mm, F.Cu at (210.1, 54.1)
- added REF**: MountingHole_3mm, MountingHole:MountingHole_3mm, F.Cu at (69.3, 133.9)
- added REF**: MountingHole_3mm, MountingHole:MountingHole_3mm, F.Cu at (69.3, 54.1)
- added REF**: MountingHole_3mm, MountingHole:MountingHole_3mm, F.Cu at (210.1, 133.9)
- J1: footprint Connector_RJ:RJ45_Connfly_DS1128-09-S8xx-S_Horizontal -> MRDT_Connectors:RJ45_Teensy
- moved J1 23.0 mm to (101.3, 63.0)
- moved Conn1 20.3 mm to (84.6, 115.1)
- moved C9 10.4 mm to (105.4, 62.5), turned to 180 degrees
- moved TP1 2.29 mm to (124.0, 67.0)
- moved C13 1.63 mm to (173.0, 98.0)
- moved R11 1.53 mm to (117.0, 65.0)
- moved C8 0.99 mm to (147.8, 104.9)
- moved R1 0.91 mm to (134.0, 100.0)
- moved C11 0.88 mm to (166.0, 99.4)
- moved TP7 0.82 mm to (148.0, 108.0)
- moved C21 0.64 mm to (183.0, 86.5)
- moved C6 0.51 mm to (139.1, 111.0)
- moved C7 0.51 mm to (143.5, 111.0)
- moved TP3 0.51 mm to (134.2, 66.0)
- moved C5 0.49 mm to (134.1, 110.0)
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Routing:
- net +12V: track 356.0 -> 440.9 mm, vias 13 -> 19
- net CS_3: track 51.0 -> 74.2 mm
- net R+: track 27.7 -> 50.3 mm
- net BSTB_3: track 34.4 -> 55.8 mm, vias 2 -> 4
- net CS_2: track 40.6 -> 57.2 mm
- net CS_1: track 41.3 -> 57.8 mm
- net R-: track 30.3 -> 46.7 mm
- net BSTA_3: track 28.4 -> 43.2 mm, vias 1 -> 3
- net Net-(C9-Pad2): track 16.5 -> 31.2 mm, vias 1 -> 0
- net T+: track 32.7 -> 45.6 mm, vias 1 -> 0
- net +3V3: track 243.9 -> 254.4 mm
- net GND: track 4.59 -> 14.5 mm, vias 4 -> 15
- net T-: track 35.7 -> 45.6 mm, vias 1 -> 0
- net BSTB_1: track 33.4 -> 42.6 mm
- net BSTC_1: track 40.8 -> 49.3 mm
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Other:
- board size 305.1 x 210.8 mm -> 239 x 160 mm

Commit message: Garrett Changes
Fixed some stray disconnected traces
Added mounting holes to schematic
Flipped ethernet port placement 180 degrees
Adjusted skew on Ethernet differential pairs
Replaced 470nf capacitor with correct 0603 ceramic capacitor (Was 470 uf and electrolytic)
Removed test points measurable directly from Teensey or Andersons
Parts:
- removed REF** (x4): MountingHole_3mm, MountingHole:MountingHole_3mm
- removed TP1, TP10, TP16, TP2, TP3, TP4, TP6, TP8, TP9: TestPoint, TestPoint:TestPoint_Pad_D2.0mm
- added H1: MountingHole, MountingHole:MountingHole_3mm, F.Cu at (210.1, 49.0)
- added H2: MountingHole, MountingHole:MountingHole_3mm, F.Cu at (84.6, 133.9)
- added H3: MountingHole, MountingHole:MountingHole_3mm, F.Cu at (84.6, 49.0)
- added H4: MountingHole, MountingHole:MountingHole_3mm, F.Cu at (210.1, 133.9)
- C15, C24: value 470 uF -> 470 nF; footprint Capacitor_THT:CP_Radial_D10.0mm_P5.00mm -> Capacitor_SMD:C_0603_1608Metric_Pad1.08x0.95mm_HandSolder
- C4: footprint Capacitor_THT:CP_Radial_D10.0mm_P5.00mm -> Capacitor_SMD:C_0603_1608Metric_Pad1.08x0.95mm_HandSolder
- U2, U4, U5: footprint DRV8329:VQFN40_RGF_TEX -> DRV8329:REE0036A-IPC_A
- moved TP11 29.6 mm to (194.6, 95.2)
- moved TP21 24.5 mm to (189.7, 58.4)
- moved R12 24.0 mm to (120.7, 107.0), turned to 90 degrees
- moved D3 18.8 mm to (120.7, 102.8), turned to -90 degrees
- moved TP23 18.7 mm to (210.6, 87.4)
- moved R11 18.2 mm to (135.1, 63.2)
- moved Conn15 17.7 mm to (129.0, 57.9)
- moved R14 16.6 mm to (130.3, 63.2)
- moved R4 15.7 mm to (140.2, 90.7), turned to 180 degrees
- moved Conn1 15.2 mm to (99.8, 116.0)
- moved J1 14.3 mm to (89.3, 55.2), turned to -90 degrees
- moved TP20 13.9 mm to (174.8, 61.0)
- moved C24 13.1 mm to (186.4, 80.3), turned to 90 degrees
- moved C9 13.0 mm to (117.1, 56.9)
- moved R38 12.8 mm to (182.6, 60.7)
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Connections:
- net BSTA_1 renamed SHA_1
- net BSTA_2 renamed SHA_2
- net BSTA_3 renamed SHA_3
- net BSTB_1 renamed SHB_1
- net BSTB_2 renamed SHB_2
- net BSTB_3 renamed SHB_3
- net BSTC_1 renamed SHC_1
- net BSTC_2 renamed SHC_2
- net BSTC_3 renamed SHC_3
Routing:
- net +3V3: track 254.4 -> 316.5 mm, vias 13 -> 16
- net GND: track 14.5 -> 73.5 mm, vias 15 -> 7
- net +12V: track 440.9 -> 401.6 mm, vias 19 -> 12
- net R+: track 50.3 -> 20.4 mm
- net R-: track 46.7 -> 20.3 mm
- net DRVOFF: track 162.1 -> 188.0 mm, vias 8 -> 6
- net CS_1: track 57.8 -> 83.3 mm
- net CS_2: track 57.2 -> 80.9 mm
- net Net-(C9-Pad2): track 31.2 -> 12.9 mm, vias 0 -> 1
- net SHA_3: track 43.2 -> 59.6 mm, vias 3 -> 2
- net nSLEEP_3: track 59.7 -> 44.7 mm, vias 3 -> 2
- net Net-(U5-AVDD): track 19.1 -> 6.00 mm
- net SHC_3: track 63.4 -> 76.3 mm
- net SHB_3: track 55.8 -> 67.2 mm, vias 4 -> 2
- net Net-(U5-CPH): track 16.1 -> 5.62 mm
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Other:
- board size 239 x 160 mm -> 132.1 x 91.4 mm

Commit message: Final changes before ordering (hopefully)
Added a pin for the ground pad in the middle of the microcontrollers so it would actually connect to ground
Also added a via to the ground pad in the middle of the microcontroller because the schematic example had some
Put vias on some other non-connected ground plane areas
Parts:
- moved C27 0.39 mm to (192.9, 66.1)
Connections:
- U2 pad 37: (no net) -> GND
- U4 pad 37: (no net) -> GND
- U5 pad 37: (no net) -> GND
Routing:
- net Net-(D2-A): track 0.00 -> 2.53 mm
- net GHA_1: track 18.5 -> 19.0 mm
- net GND: vias 7 -> 14
- net (no net): vias 3 -> 0
Changed lines of the file:
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@@
 		(tags "resistor handsolder")
 		(property "Reference" "R31"
-			(at 3.302 0 0)
+			(at -3.2004 0.1524 0)
 			(layer "F.SilkS")
 			(effects
@@
 		(placed yes)
 		(layer "F.Cu")
-		(at 192.532 66.04 90)
+		(at 192.913 66.1416 90)
 		(descr "Capacitor SMD 0603 (1608 Metric), square (rectangular) end terminal, IPC_7351 nominal with elongated pad for handsoldering. (Body size source: IPC-SM-782 page 76, https://www.pcb-3d.com/wordpress/wp-content/uploads/ipc-sm-782a_amendment_1_and_2.pdf), generated with kicad-footprint-generator")
 		(tags "capacitor handsolder")
@@
 		(tags "PDRV8329AREER ")
 		(property "Reference" "U4"
-			(at 0.127 -2.7178 0)
+			(at -4.3434 -0.2286 0)
 			(unlocked yes)
 			(layer "F.SilkS")
@@
 			(layer "F.Fab")
 		)
-		(fp_text user "Designator295"
-			(at -0.0254 -4.0894 0)
-			(unlocked yes)
-			(layer "F.SilkS")
-			(effects
-				(font
-					(size 1 1)
-					(thickness 0.15)
-				)
-			)
-		)
 		(fp_text user "${REFERENCE}"
 			(at 0 0 0)
@@
 			(size 2.799999 3.8)
 			(layers "F.Cu" "F.Mask")
+			(net 2 "GND")
+			(pinfunction "Ground")
+			(pintype "power_out")
 		)
 	)
@@
 		(tags "PDRV8329AREER ")
 		(property "Reference" "U5"
-			(at -0.144 -3.1496 90)
+			(at -0.3218 4.2164 90)
 			(unlocked yes)
 			(layer "F.SilkS")
@@
 			(layer "F.Fab")
 		)
-		(fp_text user "Designator295"
-			(at -3.2512 -4.7244 90)
-			(unlocked yes)
-			(layer "F.SilkS")
-			(effects
-				(font
-					(size 1 1)
-					(thickness 0.15)
-				)
-			)
-		)
 		(fp_text user "${REFERENCE}"
 			(at 0 0 90)
@@
 			(size 2.799999 3.8)
 			(layers "F.Cu" "F.Mask")
+			(net 2 "GND")
+			(pinfunction "ground")
+			(pintype "power_out")
 		)
 	)
@@
 		(tags "PDRV8329AREER ")
 		(property "Reference" "U2"
-			(at -0.0762 -3.2766 0)
+			(at -0.0762 -3.9878 0)
 			(unlocked yes)
 			(layer "F.SilkS")
@@
 			(layer "F.Fab")
 		)
-		(fp_text user "Designator295"
-			(at 0.127 3.7084 0)
-			(unlocked yes)
-			(layer "F.SilkS")
-			(effects
-				(font
-					(size 1 1)
-					(thickness 0.15)
-				)
-			)
-		)
 		(fp_text user "${REFERENCE}"
 			(at 0 0 0)
@@
 			(size 2.799999 3.8)
 			(layers "F.Cu" "F.Mask")
+			(net 2 "GND")
+			(pinfunction "Ground")
+			(pintype "power_out")
 		)
 	)
@@
 		(layer "Edge.Cuts")
 	)
-	(via
-		(at 179.324 104.394)
-		(size 0.6)
-		(drill 0.3)
-		(layers "F.Cu" "B.Cu")
-		(net 0)
-	)
-	(via
-		(at 184.404 72.373)
-		(size 0.6)
-		(drill 0.3)
-		(layers "F.Cu" "B.Cu")
-		(net 0)
-	)
-	(via
-		(at 139.319 103.632)
-		(size 0.6)
-		(drill 0.3)
-		(layers "F.Cu" "B.Cu")
-		(net 0)
-	)
 	(segment
 		(start 168.937962 104.194)
@@
 	)
 	(via
+		(at 184.404 72.373)
+		(size 0.6)
+		(drill 0.3)
+		(layers "F.Cu" "B.Cu")
+		(net 2)
+	)
+	(via
+		(at 199.8218 77.0128)
+		(size 0.6)
+		(drill 0.3)
+		(layers "F.Cu" "B.Cu")
+		(free yes)
+		(net 2)
+	)
+	(via
 		(at 176.276 99.314)
 		(size 0.6)
@@
 	)
 	(via
+		(at 139.319 103.632)
+		(size 0.6)
+		(drill 0.3)
+		(layers "F.Cu" "B.Cu")
+		(net 2)
+	)
+	(via
 		(at 133.604 102.362)
 		(size 0.6)
@@
 	)
 	(via
+		(at 128.8288 107.6452)
+		(size 0.6)
+		(drill 0.3)
+		(layers "F.Cu" "B.Cu")
+		(free yes)
+		(net 2)
+	)
+	(via
 		(at 145.034 102.616)
 		(size 0.6)
@@
 	)
 	(via
+		(at 183.8452 83.3882)
+		(size 0.6)
+		(drill 0.3)
+		(layers "F.Cu" "B.Cu")
+		(free yes)
+		(net 2)
+	)
+	(via
 		(at 169.418 103.378)
 		(size 0.6)
@@
 		(net 2)
 	)
+	(via
+		(at 161.798 116.0272)
+		(size 0.6)
+		(drill 0.3)
+		(layers "F.Cu" "B.Cu")
+		(free yes)
+		(net 2)
+	)
+	(via
+		(at 179.324 104.394)
+		(size 0.6)
+		(drill 0.3)
+		(layers "F.Cu" "B.Cu")
+		(net 2)
+	)
 	(segment
 		(start 134.228499 104.632001)
@@
 	)
 	(segment
-		(start 192.6325 65.278)
-		(end 192.532 65.1775)
-		(width 0.508)
-		(layer "F.Cu")
-		(net 32)
-	)
-	(segment
-		(start 194.31 65.278)
-		(end 192.6325 65.278)
+		(start 203.57825 63.12175)
+		(end 204.5915 64.135)
 		(width 0.508)
 		(layer "F.Cu")
@@
 	)
 	(segment
-		(start 203.57825 63.12175)
-		(end 204.5915 64.135)
-		(width 0.508)
+		(start 192.4304 65.2791)
+		(end 192.913 65.2791)
+		(width 0.2)
 		(layer "F.Cu")
 		(net 32)
@@
 	)
 	(segment
-		(start 186.907033 70.973)
-		(end 186.907033 70.802467)
-		(width 0.2)
-		(layer "F.Cu")
-		(net 32)
-	)
-	(segment
 		(start 203.475 62.738)
 		(end 203.475 59.3905)
@@
 	)
 	(segment
-		(start 186.907033 70.802467)
-		(end 192.532 65.1775)
+		(start 186.907033 70.973)
+		(end 186.837 70.973)
 		(width 0.2)
 		(layer "F.Cu")
@@
 	)
 	(segment
-		(start 186.907033 70.973)
-		(end 186.837 70.973)
-		(width 0.2)
+		(start 192.9141 65.278)
+		(end 192.913 65.2791)
+		(width 0.508)
 		(layer "F.Cu")
 		(net 32)
@@
 	)
 	(segment
+		(start 186.907033 70.802467)
+		(end 192.4304 65.2791)
+		(width 0.2)
+		(layer "F.Cu")
+		(net 32)
+	)
+	(segment
+		(start 186.907033 70.973)
+		(end 186.907033 70.802467)
+		(width 0.2)
+		(layer "F.Cu")
+		(net 32)
+	)
+	(segment
+		(start 194.31 65.278)
+		(end 192.9141 65.278)
+		(width 0.508)
+		(layer "F.Cu")
+		(net 32)
+	)
+	(segment
 		(start 203.57825 63.12175)
 		(end 203.475 63.0185)
@@
 	)
 	(segment
-		(start 192.1775 66.9025)
+		(start 192.0759 67.0041)
 		(end 190.246 68.834)
 		(width 0.508)
@@
 	)
 	(segment
-		(start 192.532 66.9025)
-		(end 192.1775 66.9025)
-		(width 0.508)
+		(start 186.907033 71.372999)
+		(end 187.707001 71.372999)
+		(width 0.2)
 		(layer "F.Cu")
 		(net 33)
 	)
 	(segment
-		(start 186.907033 71.372999)
-		(end 187.707001 71.372999)
-		(width 0.2)
+		(start 192.913 67.0041)
+		(end 192.0759 67.0041)
+		(width 0.508)
 		(layer "F.Cu")
 		(net 33)
@@
 	)
 	(segment
+		(start 105.273 106.5345)
+		(end 105.273 104.004)
+		(width 0.254)
+		(layer "F.Cu")
+		(net 39)
+	)
+	(segment
 		(start 120.65 103.632)
 		(end 120.65 106.125)
@@
 	)
 	(segment
+		(start 137.922 106.138033)
+		(end 137.922 106.4006)
+		(width 0.2)
+		(layer "F.Cu")
+		(net 80)
+	)
+	(segment
+		(start 137.919 106.135033)
+		(end 137.919 105.8448)
+		(width 0.2)
+		(layer "F.Cu")
+		(net 80)
+	)
+	(segment
 		(start 131.14 112.954)
 		(end 123.6235 112.954)
@@
 	)
 	(segment
+		(start 137.919 105.8448)
+		(end 137.922 105.8418)
+		(width 0.2)
+		(layer "F.Cu")
+		(net 80)
+	)
+	(segment
 		(start 134.600016 109.493984)
 		(end 131.14 112.954)
@@
 	)
 	(segment
+		(start 137.919 106.135033)
+		(end 137.922 106.138033)
+		(width 0.2)
+		(layer "F.Cu")
+		(net 80)
+	)
+	(segment
 		(start 135.89 109.474)
 		(end 131.4685 113.8955)
@@
 	)
 	(segment
-		(start 186.203999 70.369969)
-		(end 186.203999 70.013173)
-		(width 0.2)
+		(start 192.3034 63.7032)
+		(end 191.481586 64.525014)
+		(width 0.508)
 		(layer "F.Cu")
 		(net 97)
 	)
 	(segment
-		(start 192.00149 64.186)
-		(end 191.481586 64.705904)
+		(start 196.9595 65.142)
+		(end 195.5207 63.7032)
 		(width 0.508)
 		(layer "F.Cu")
@@
 	)
 	(segment
-		(start 196.9595 65.142)
-		(end 196.0035 64.186)
+		(start 191.481586 64.525014)
+		(end 191.481586 64.735586)
 		(width 0.508)
 		(layer "F.Cu")
@@
 	)
 	(segment
-		(start 186.203999 70.013173)
-		(end 191.877172 64.34)
+		(start 186.203999 70.369969)
+		(end 186.203999 70.013173)
 		(width 0.2)
 		(layer "F.Cu")
@@
 	)
 	(segment
+		(start 195.5207 63.7032)
+		(end 192.3034 63.7032)
+		(width 0.508)
+		(layer "F.Cu")
+		(net 97)
+	)
+	(segment
 		(start 186.203999 70.582838)
 		(end 186.200237 70.5866)
@@
 	)
 	(segment
-		(start 196.0035 64.186)
-		(end 192.00149 64.186)
-		(width 0.508)
+		(start 186.203999 70.013173)
+		(end 191.481586 64.735586)
+		(width 0.2)
 		(layer "F.Cu")
 		(net 97)
