File: Hardware/BrushlessGimbalController_Hardware/BrushlessGimbalController_Hardware.kicad_sch (KiCad schematic)
At the start: 103 parts, among them J1 8P8C_LED_Shielded, Q1 NMOS, Q10 NMOS, Q11 NMOS, Q12 NMOS, Q13 NMOS, Q14 NMOS, Q15 NMOS, Q16 NMOS, Q17 NMOS, Q18 NMOS, Q2 NMOS, Q3 NMOS, Q4 NMOS, Q5 NMOS, Q6 NMOS, Q7 NMOS, Q8 NMOS, Q9 NMOS, U3 Teensy4.1_DEV-16771, U5 OKI

Commit message: Un-fucking files pt.2
Parts:
- removed C29, C30: 0.1uf, symbol Device:C
- removed C31: 1 uF, symbol Device:C
- removed C32: 60uF, symbol Device:C
- removed Conn1: AndersonPP, symbol MRDT_Connectors:AndersonPP
- removed Conn10: Molex_SL_04, symbol MRDT_Connectors:Molex_SL_04
- removed D6, D7, D8: LED, symbol Device:LED
- removed R37: 280, symbol Device:R
- removed R38, R39: 47k, symbol Device:R
- removed U3: Teensy4.1_DEV-16771, MODULE_DEV-16771, symbol MRDT_Shields:Teensy4.1_DEV-16771
- removed U5: OKI, symbol MRDT_Devices:OKI
- removed U6, U7: ~, symbol MRDT_Devices:DRV8239
- added C1: 0.1uF, symbol Device:C
- added C2, C3: 10 uF, symbol Device:C
- added C4: 60uF, symbol Device:C
- added Conn1: Molex_SL_04, symbol MRDT_Connectors:Molex_SL_04
- added Conn10: AndersonPP, symbol MRDT_Connectors:AndersonPP
- added unit 4 of Conn2
- added unit 1 of Conn2
- added D3, D4, D5: LED, symbol Device:LED
- added R1, R2: 47k, symbol Device:R
- added R3: 70, symbol Device:R
- added U1: Teensy4.1_DEV-16771, MODULE_DEV-16771, symbol MRDT_Shields:Teensy4.1_DEV-16771
- added U2: OKI, symbol MRDT_Devices:OKI
- added U3: ~, QFN, symbol MRDT_Devices:DRV8239
- added U5: ~, symbol MRDT_Devices:DRV8239
- C10: value 1 uF -> 20 uF
- C11: value 20 uF -> 10uf
- C12: value 0.1 uF -> 10uf
- C13: value 1uf -> 10uf
- C14: value 0.1uf -> 470 nF
- C15: value 0.1uf -> 470 uF
- C16: value 0.1 uF -> 470 uF
- C17: value 20 uF -> 1uf
- C18: value 10uf -> 0.1uf
- C19: value 470 uF -> 0.1uf
- C23: value 1 uF -> 0.1uf
- C24: value 0.1 uF -> 0.1uf
- C25: value 20 uF -> 0.1uf
- C26: value 10uf -> 1 uF
- C27: value 470 uF -> 1 uF
- C28: value 0.1uf -> 1 uF
- C5: value 0.1uF -> 0.1 uF
- C6, C7: value 10 uF -> 0.1 uF
- C8: value 10uf -> 20 uF
- C9: value 470 nF -> 20 uF
- R10, R11, R12, R5, R6, R9: value 47 -> R
- R13, R15: value 0.64 -> 280
- R14: value R -> 280
- R16, R17, R18: value 47 -> 0.64
- R22, R32, R33, R34, R35: value R -> 47
- R23: value 0.64 -> 47
- R30: value 400K -> 47
- R31: value 1K -> 47
- R36: value 280 -> 47
- R4: value 280 -> 4.7k
- R7: value 70 -> 400K
- R8: value 4.7k -> 1K
- U4: footprint QFN -> (none)
Connections:
- net +12V: now also C10.2, C5.2, C6.2, C7.2, C8.2, C9.2, R4.1, C2.1, C4.1, Conn2.4 (PV+), U2.1 (Vi), U3.5 (PVDD), U5.5 (PVDD); no longer C11.2, C12.2, C16.2, C17.2, C24.2, C25.2, C6.1, R8.1
- net +3.3V: now also U1.3.3V_1 (3.3V), U1.3.3V_2 (3.3V), U1.3.3V_3 (3.3V)
- net +3V3: now also R11.2, R13.2, R14.2, R15.2, R7.2, R9.2, C3.1, Conn1.2, R1.1, R2.2, R3.1, U2.3 (Vo), U3.1 (CSAREF), U3.30 (INLC), U3.31 (INLB), U3.32 (INLA), U5.1 (CSAREF), U5.30 (INLC), U5.31 (INLB), U5.32 (INLA); no longer C7.1, R30.2, R32.2, R34.2, R36.2, R4.2, R7.1
- net BSTA: now also C17.2, C18.2, C19.1, Conn2.1, Q15.3 (S), Q16.1 (D), Conn10.1, U3.10 (SHA), U5.10 (SHA); no longer C13.2, C20.2, C28.1, Conn6.1, Q11.3 (S), Q12.1 (D)
- net BSTB: now also C20.2, C22.2, Conn3.1, Conn5.1, Q11.3 (S), Q12.1 (D), U3.14 (SHB), U5.14 (SHB); no longer C14.2, Conn2.1, Conn4.1, Q13.3 (S), Q14.1 (D)
- net BSTC: now also C23.2, C24.2, C25.2, Conn4.1, Conn6.1, Q13.3 (S), Q14.1 (D), U3.18 (SHC), U5.18 (SHC); no longer C15.2, C22.2, Conn3.1, Conn5.1, Q15.3 (S), Q16.1 (D)
- net CS: now also R16.2, R17.2, U3.21 (LSS), U3.22 (SP); no longer R13.2, R15.2
- net CS_1: now also Q16.3 (S); no longer Q12.3 (S)
- net CS_3: now also Q12.3 (S); no longer Q16.3 (S)
- net DRVOFF: now also U1.14 (A0), U3.24 (DRVOFF), U5.24 (DRVOFF)
- net GHA: now also R19.1, U3.11 (GHA), U5.11 (GHA); no longer R5.1
- net GHB: now also R21.1, R25.1, R29.1, R33.1, R35.1, U3.15 (GLB), U5.15 (GLB); no longer R16.1, R20.1, R24.1, R28.1, R9.1
- net GHC: now also R23.1, R27.1, R31.1, U3.19 (GHC), U5.19 (GHC); no longer R11.1, R18.1, R26.1
- net GLA: now also R20.1, U3.12 (GLA), U5.12 (GLA); no longer R6.1
- net GLB: now also R22.1, R26.1, R30.1, R34.1, R36.1, U3.15 (GLB), U5.15 (GLB); no longer R10.1, R17.1, R21.1, R25.1, R29.1
- net GLC: now also R24.1, R28.1, R32.1, U3.20 (GLC), U5.20 (GLC); no longer R12.1, R19.1, R27.1
- net GND: now also C11.2, C12.2, C13.2, C26.1, C27.1, C28.1, C6.1, C7.1, C8.1, C9.1, R10.1, R12.1, R16.1, R17.1, R18.1, R5.1, R6.1, R8.1, C1.1, C2.2, C3.2, C4.2, Conn1.1, Conn2.1 (GND), U1.GND1 (GND), U1.GND2 (GND), U1.GND3 (GND), U1.GND4 (GND), U1.GND5 (GND), U1.USB_GND1 (USB_GND), U1.USB_GND2 (USB_GND), U2.2 (GND), U3.23 (SN), U3.25 (AGND), U3.3 (DT), U3.33 (CSAGAIN), U3.4 (GND), U5.23 (SN), U5.33 (CSAGAIN), U5.4 (GND); no longer C11.1, C12.1, C16.1, C17.1, C18.2, C23.1, C24.1, C25.1, C26.2, C6.2, C7.2, C8.2, R13.1, R14.1, R15.1, R22.1, R23.1, R31.1, R33.1, R35.1, U4.25 (AGND), U4.3 (DT)
- net LED: now also U1.LED
- net PWM A (1): now also U1.1 (TX1), U3.29 (INHA); no longer U4.29 (INHA)
- net PWM A (2): now also U4.29 (INHA), U1.4 (BCLK2)
- net PWM A (3): now also U1.7 (RX2), U5.29 (INHA)
- net PWM B (1): now also U1.2 (OUT2), U3.28 (INHB); no longer U4.28 (INHB)
- net PWM B (2): now also U4.28 (INHB), U1.5 (IN2)
- net PWM B (3): now also U1.8 (TX2), U5.28 (INHB)
- net PWM C (1): now also U1.3 (LRCLK2), U3.27 (INHC); no longer U4.27 (INHC)
- net PWM C (2): now also U4.27 (INHC), U1.6 (OUT1D)
- net PWM C (3): now also U1.9 (OUT1C), U5.27 (INHC)
- net SCK: now also U1.27 (A13)
- net SCL: now also Conn1.4, R1.2, U1.24 (A10)
- net SDA: now also Conn1.3, R2.1, U1.25 (A11)
- net SO (1): now also U1.41 (A17), U3.2 (SO); no longer U4.2 (SO)
- net SO (2): now also U4.2 (SO), U1.40 (A16)
- net SO (3): now also U1.39 (A15), U5.2 (SO)
- net nFAULT (1): now also D5.1 (K), U1.32 (OUT1B), U3.35 (nFAULT); no longer U4.35 (nFAULT)
- net nFAULT (2): now also U4.35 (nFAULT), D3.1 (K), U1.30 (CRX3)
- net nFAULT (3): now also D4.1 (K), U1.31 (CTX3), U5.35 (nFAULT)
- net nSLEEP (1): now also U1.28 (RX7), U3.34 (nSLEEP); no longer U4.34 (nSLEEP)
- net nSLEEP (2): now also U4.34 (nSLEEP), U1.29 (TX7)
- net nSLEEP (3): now also U1.26 (A12), U5.34 (nSLEEP)
- net at Q11.2 (G): now also R29.2; no longer R20.2
- net at U4.26 (AVDD): now also C26.2; no longer C10.2
- net at Q1.2 (G): now also R21.2; no longer R9.2
- net at C13.1: now also U5.8 (GVDD); no longer U4.9 (BSTA)
- net at J1.1: now also U1.T+
- net at J1.2, J1.5: now also C1.2; no longer C5.2
- net at J1.3: now also U1.T-
- net at J1.4: now also U1.R+
- net at J1.6: now also U1.R-
- net at U4.13 (BSTA): now also C21.1; no longer C14.1
- net at U4.17 (BSTC): now also C24.1; no longer C15.1
- net at U4.6 (CPL): now also C15.1; no longer C9.1
- net at U4.7 (CPH): now also C15.2; no longer C9.2
- net at U4.8 (GVDD): now also C12.1; no longer C8.1
- net at R18.2: now also U5.21 (LSS), U5.22 (SP); no longer Q9.2 (G)
- net at R6.2: now also U5.3 (DT); no longer Q6.2 (G)
- net at Q12.2 (G): now also R30.2; no longer R21.2
- net at Q10.2 (G): now also R28.2; no longer R19.2
- net at Q7.2 (G): now also R25.2; no longer R16.2
- net at Q15.2 (G): now also R33.2; no longer R26.2
- net at Q17.2 (G): now also R35.2; no longer R28.2
- net at C28.2: now also U3.26 (AVDD)
- net at R22.2: now also Q2.2 (G)
- net at R24.2: now also Q4.2 (G); no longer Q13.2 (G)
- net at C22.1: now also U5.13 (BSTA)
- net at R5.2: now also U4.3 (DT); no longer Q5.2 (G)
- net at C27.2: now also U5.26 (AVDD)
- net at D2.2 (A): now also R4.2; no longer R8.2
- net at Q14.2 (G): now also R32.2; no longer R25.2
- net at Q18.2 (G): now also R36.2; no longer R29.2
- net at R27.2: now also Q9.2 (G); no longer Q16.2 (G)
- net at D1.2 (A): now also R3.2; no longer R7.2
- net at Q8.2 (G): now also R26.2; no longer R17.2
- net at R10.2: now also R9.1, U4.36 (VDSLVL); no longer Q2.2 (G)
- net at C20.1: now also U3.13 (BSTA)
- net at C19.2: now also U5.9 (BSTA)
- net at C18.1: now also U4.9 (BSTA)
- net at Q3.2 (G): now also R23.2; no longer R11.2
- net at R12.2: now also R11.1, U5.36 (VDSLVL); no longer Q4.2 (G)
- new net: C25.1, U5.17 (BSTC)
- new net: C16.1, U5.6 (CPL)
- new net: C16.2, U5.7 (CPH)
- new net: C11.1, U3.8 (GVDD)
- new net: D4.2 (A), R14.1
- new net: C23.1, U3.17 (BSTC)
- new net: R7.1, R8.2, U3.36 (VDSLVL)
- new net: D3.2 (A), R13.1
- new net: Q5.2 (G), R19.2
- new net: D5.2 (A), R15.1
- new net: C14.1, U3.6 (CPL)
- new net: C14.2, U3.7 (CPH)
- new net: Q13.2 (G), R31.2
- new net: Q6.2 (G), R20.2
- new net: Q16.2 (G), R34.2
- new net: C17.1, U3.9 (BSTA)

Commit message: Layout Ready For Review
Added all of the traces and ground planes and vias and things
Parts:
- removed C1: 0.1uF, symbol Device:C
- removed C4: 60uF, symbol Device:C
- removed Conn10, Conn3, Conn4, Conn5, Conn6, Conn7, Conn8, Conn9: AndersonPP, symbol MRDT_Connectors:AndersonPP
- removed unit 5 of Conn2
- added C18: 100uF, Capacitor_THT:C_Radial_D6.3mm_H5.0mm_P2.50mm, symbol Device:C_Polarized
- added C9: 0.1uF, Capacitor_SMD:C_0603_1608Metric_Pad1.08x0.95mm_HandSolder, symbol Device:C
- added Conn2, Conn3, Conn4: Molex_SL_03, Connector_Molex:Molex_SL_171971-0003_1x03_P2.54mm_Vertical, symbol MRDT_Connectors:Molex_SL_03
- added R1: 10K, Resistor_SMD:R_0603_1608Metric_Pad0.98x0.95mm_HandSolder, symbol Device:R
- added R15, R33, R5: 200K, Resistor_SMD:R_0603_1608Metric_Pad0.98x0.95mm_HandSolder, symbol Device:R
- added TP1, TP10, TP11, TP12, TP13, TP14, TP15, TP16, TP17, TP18, TP19, TP2, TP20, TP21, TP22, TP23, TP24, TP3, TP4, TP5, TP6, TP7, TP8, TP9: TestPoint, TestPoint:TestPoint_Pad_D2.0mm, symbol Connector:TestPoint
- C1: renamed from C5; footprint (none) -> Capacitor_SMD:C_0603_1608Metric_Pad1.08x0.95mm_HandSolder
- C10: renamed from C2; footprint (none) -> Capacitor_SMD:C_0603_1608Metric_Pad1.08x0.95mm_HandSolder
- C11: renamed from C6; footprint (none) -> Capacitor_SMD:C_0603_1608Metric_Pad1.08x0.95mm_HandSolder
- C12: renamed from C3; footprint (none) -> Capacitor_SMD:C_0603_1608Metric_Pad1.08x0.95mm_HandSolder
- C13: renamed from C9; value 20 uF -> 22 uF; footprint (none) -> Capacitor_THT:CP_Radial_D5.0mm_P2.00mm
- C14: renamed from C12; footprint (none) -> Capacitor_SMD:C_0603_1608Metric_Pad1.08x0.95mm_HandSolder
- C15: footprint (none) -> Capacitor_THT:CP_Radial_D10.0mm_P5.00mm
- C16: renamed from C18; value 0.1uf -> 1uf; footprint (none) -> Capacitor_SMD:C_0603_1608Metric_Pad1.08x0.95mm_HandSolder
- C17: renamed from C21; value 0.1uf -> 1uf; footprint (none) -> Capacitor_SMD:C_0603_1608Metric_Pad1.08x0.95mm_HandSolder
- C19: renamed from C24; value 0.1uf -> 1uf; footprint (none) -> Capacitor_SMD:C_0603_1608Metric_Pad1.08x0.95mm_HandSolder
- C2: renamed from C8; value 20 uF -> 22 uF; footprint (none) -> Capacitor_THT:CP_Radial_D5.0mm_P2.00mm
- C20: renamed from C26; footprint (none) -> Capacitor_SMD:C_0603_1608Metric_Pad1.08x0.95mm_HandSolder
- C21: renamed from C7; footprint (none) -> Capacitor_SMD:C_0603_1608Metric_Pad1.08x0.95mm_HandSolder
- C22: renamed from C10; value 20 uF -> 22 uF; footprint (none) -> Capacitor_THT:CP_Radial_D5.0mm_P2.00mm
- C23: renamed from C13; footprint (none) -> Capacitor_SMD:C_0603_1608Metric_Pad1.08x0.95mm_HandSolder
- C24: renamed from C16; footprint (none) -> Capacitor_THT:CP_Radial_D10.0mm_P5.00mm
- C25: renamed from C19; value 0.1uf -> 1uf; footprint (none) -> Capacitor_SMD:C_0603_1608Metric_Pad1.08x0.95mm_HandSolder
- C26: renamed from C22; value 0.1uf -> 1uf; footprint (none) -> Capacitor_SMD:C_0603_1608Metric_Pad1.08x0.95mm_HandSolder
- C27: renamed from C25; value 0.1uf -> 1uf; footprint (none) -> Capacitor_SMD:C_0603_1608Metric_Pad1.08x0.95mm_HandSolder
- C28: renamed from C27; footprint (none) -> Capacitor_SMD:C_0603_1608Metric_Pad1.08x0.95mm_HandSolder
- C3: renamed from C11; footprint (none) -> Capacitor_SMD:C_0603_1608Metric_Pad1.08x0.95mm_HandSolder
- C4: renamed from C14; footprint (none) -> Capacitor_THT:CP_Radial_D10.0mm_P5.00mm
- C5: renamed from C17; footprint (none) -> Capacitor_SMD:C_0603_1608Metric_Pad1.08x0.95mm_HandSolder
- C6: renamed from C20; value 0.1uf -> 1uf; footprint (none) -> Capacitor_SMD:C_0603_1608Metric_Pad1.08x0.95mm_HandSolder
- C7: renamed from C23; value 0.1uf -> 1uf; footprint (none) -> Capacitor_SMD:C_0603_1608Metric_Pad1.08x0.95mm_HandSolder
- C8: renamed from C28; footprint (none) -> Capacitor_SMD:C_0603_1608Metric_Pad1.08x0.95mm_HandSolder
- Conn1: renamed from Conn2; footprint (none) -> MRDT_Connectors:Square_Anderson_2_H_Side_By_Side
- Conn15: renamed from Conn1; footprint (none) -> MRDT_Connectors:MOLEX_SL_04_Vertical
- D1: renamed from D5; value LED -> GREEN; footprint (none) -> LED_SMD:LED_0603_1608Metric_Pad1.05x0.95mm_HandSolder
- D2: renamed from D1; value LED -> GREEN; footprint (none) -> LED_SMD:LED_0603_1608Metric_Pad1.05x0.95mm_HandSolder
- D3: renamed from D2; value LED -> GREEN; footprint (none) -> LED_SMD:LED_0603_1608Metric_Pad1.05x0.95mm_HandSolder
- D4: renamed from D3; value LED -> GREEN; footprint (none) -> LED_SMD:LED_0603_1608Metric_Pad1.05x0.95mm_HandSolder
- D5: renamed from D4; value LED -> GREEN; footprint (none) -> LED_SMD:LED_0603_1608Metric_Pad1.05x0.95mm_HandSolder
- J1: footprint (none) -> Connector_RJ:RJ45_Connfly_DS1128-09-S8xx-S_Horizontal
- Q1, Q10, Q17, Q18, Q2, Q3, Q4, Q5, Q6, Q7, Q8, Q9: footprint (none) -> Package_TO_SOT_SMD:SOT-23-3
- Q11: renamed from Q15; footprint (none) -> Package_TO_SOT_SMD:SOT-23-3
- Q12: renamed from Q16; footprint (none) -> Package_TO_SOT_SMD:SOT-23-3
- Q13: renamed from Q11; footprint (none) -> Package_TO_SOT_SMD:SOT-23-3
- Q14: renamed from Q12; footprint (none) -> Package_TO_SOT_SMD:SOT-23-3
- Q15: renamed from Q13; footprint (none) -> Package_TO_SOT_SMD:SOT-23-3
- Q16: renamed from Q14; footprint (none) -> Package_TO_SOT_SMD:SOT-23-3
- R10: value R -> 1K; footprint (none) -> Resistor_SMD:R_0603_1608Metric_Pad0.98x0.95mm_HandSolder
- R11: renamed from R2; value 47k -> 4.7K; footprint (none) -> Resistor_SMD:R_0603_1608Metric_Pad0.98x0.95mm_HandSolder
- R12: renamed from R4; footprint (none) -> Resistor_SMD:R_0603_1608Metric_Pad0.98x0.95mm_HandSolder
- R13: value 280 -> 300; footprint (none) -> Resistor_SMD:R_0603_1608Metric_Pad0.98x0.95mm_HandSolder
- R14: renamed from R1; value 47k -> 4.7K; footprint (none) -> Resistor_SMD:R_0603_1608Metric_Pad0.98x0.95mm_HandSolder
- R16: renamed from R17; value 0.64 -> 0.1; footprint (none) -> Resistor_SMD:R_2816_7142Metric_Pad3.20x4.45mm_HandSolder
- R17: renamed from R19; value 47 -> 30; footprint (none) -> Resistor_SMD:R_0603_1608Metric_Pad0.98x0.95mm_HandSolder
- R18: renamed from R20; value 47 -> 30; footprint (none) -> Resistor_SMD:R_0603_1608Metric_Pad0.98x0.95mm_HandSolder
- R19: renamed from R21; value 47 -> 30; footprint (none) -> Resistor_SMD:R_0603_1608Metric_Pad0.98x0.95mm_HandSolder
- R2: renamed from R7; value 400K -> 402K; footprint (none) -> Resistor_SMD:R_0603_1608Metric_Pad0.98x0.95mm_HandSolder
- R20: renamed from R22; value 47 -> 30; footprint (none) -> Resistor_SMD:R_0603_1608Metric_Pad0.98x0.95mm_HandSolder
- R21: renamed from R23; value 47 -> 30; footprint (none) -> Resistor_SMD:R_0603_1608Metric_Pad0.98x0.95mm_HandSolder
- R22: renamed from R24; value 47 -> 30; footprint (none) -> Resistor_SMD:R_0603_1608Metric_Pad0.98x0.95mm_HandSolder
- R23: renamed from R6; value R -> 10K; footprint (none) -> Resistor_SMD:R_0603_1608Metric_Pad0.98x0.95mm_HandSolder
- R24: renamed from R25; value 47 -> 30; footprint (none) -> Resistor_SMD:R_0603_1608Metric_Pad0.98x0.95mm_HandSolder
- R25: renamed from R26; value 47 -> 30; footprint (none) -> Resistor_SMD:R_0603_1608Metric_Pad0.98x0.95mm_HandSolder
- R26: renamed from R27; value 47 -> 30; footprint (none) -> Resistor_SMD:R_0603_1608Metric_Pad0.98x0.95mm_HandSolder
- R27: renamed from R28; value 47 -> 30; footprint (none) -> Resistor_SMD:R_0603_1608Metric_Pad0.98x0.95mm_HandSolder
- R28: renamed from R33; value 47 -> 30; footprint (none) -> Resistor_SMD:R_0603_1608Metric_Pad0.98x0.95mm_HandSolder
- R29: renamed from R34; value 47 -> 30; footprint (none) -> Resistor_SMD:R_0603_1608Metric_Pad0.98x0.95mm_HandSolder
- R3: renamed from R8; footprint (none) -> Resistor_SMD:R_0603_1608Metric_Pad0.98x0.95mm_HandSolder
- R30: renamed from R11; value R -> 402K; footprint (none) -> Resistor_SMD:R_0603_1608Metric_Pad0.98x0.95mm_HandSolder
- R31: renamed from R12; value R -> 1K; footprint (none) -> Resistor_SMD:R_0603_1608Metric_Pad0.98x0.95mm_HandSolder
- R32: renamed from R14; value 280 -> 300; footprint (none) -> Resistor_SMD:R_0603_1608Metric_Pad0.98x0.95mm_HandSolder
- R34: renamed from R29; value 47 -> 30; footprint (none) -> Resistor_SMD:R_0603_1608Metric_Pad0.98x0.95mm_HandSolder
- R35: renamed from R30; value 47 -> 30; footprint (none) -> Resistor_SMD:R_0603_1608Metric_Pad0.98x0.95mm_HandSolder
- R36: renamed from R31; value 47 -> 30; footprint (none) -> Resistor_SMD:R_0603_1608Metric_Pad0.98x0.95mm_HandSolder
- R37: renamed from R32; value 47 -> 30; footprint (none) -> Resistor_SMD:R_0603_1608Metric_Pad0.98x0.95mm_HandSolder
- R38: renamed from R18; value 0.64 -> 0.1; footprint (none) -> Resistor_SMD:R_2816_7142Metric_Pad3.20x4.45mm_HandSolder
- R39: renamed from R35; value 47 -> 30; footprint (none) -> Resistor_SMD:R_0603_1608Metric_Pad0.98x0.95mm_HandSolder
- R4: renamed from R15; value 280 -> 300; footprint (none) -> Resistor_SMD:R_0603_1608Metric_Pad0.98x0.95mm_HandSolder
- R40: renamed from R36; value 47 -> 30; footprint (none) -> Resistor_SMD:R_0603_1608Metric_Pad0.98x0.95mm_HandSolder
- R6: renamed from R16; value 0.64 -> 0.1; footprint (none) -> Resistor_SMD:R_2816_7142Metric_Pad3.20x4.45mm_HandSolder
- R7: renamed from R5; value R -> 10K; footprint (none) -> Resistor_SMD:R_0603_1608Metric_Pad0.98x0.95mm_HandSolder
- R8: renamed from R3; value 70 -> 100; footprint (none) -> Resistor_SMD:R_0603_1608Metric_Pad0.98x0.95mm_HandSolder
- R9: value R -> 402K; footprint (none) -> Resistor_SMD:R_0603_1608Metric_Pad0.98x0.95mm_HandSolder
- U1: footprint MODULE_DEV-16771 -> MRDT_Shields:Teensy_4_1
- U2: renamed from U3; footprint QFN -> DRV8329:VQFN40_RGF_TEX
- U3: renamed from U2; footprint (none) -> Converter_DCDC:Converter_DCDC_Murata_OKI-78SR_Horizontal
- U4, U5: footprint (none) -> DRV8329:VQFN40_RGF_TEX
Connections:
- net +3.3V is gone; now on net +3V3: U1.3.3V_1 (3.3V), U1.3.3V_2 (3.3V), U1.3.3V_3 (3.3V)
- net +12V: now also Conn1.2 (PV+), C18.1, TP8.1; no longer Conn1.4 (PV+)
- net +3V3: now also Conn15.4, R11.1, R14.2; no longer Conn15.2, R11.2, R14.1
- net CS_1: now also Q2.3 (S), Q6.3 (S), R6.2, U2.21 (LSS), U2.22 (SP), TP7.1; no longer Q12.3 (S), Q8.3 (S)
- net CS_2: now also Q12.3 (S), Q8.3 (S), R16.2, U4.21 (LSS), U4.22 (SP), TP12.1; no longer Q18.3 (S)
- net CS_3: now also Q18.3 (S), R38.2, U5.21 (LSS), U5.22 (SP), TP21.1
- net DRVOFF: now also TP3.1
- net GND: now also U4.25 (AGND), U5.25 (AGND), C18.2, C9.1, R1.1, R15.2, R33.2, R5.2, TP9.1; no longer U2.3 (DT), U2.33 (CSAGAIN), U4.33 (CSAGAIN), U5.33 (CSAGAIN)
- net SCL: now also Conn15.2, R14.1, U1.19 (A5), TP2.1; no longer Conn15.4, R14.2, U1.24 (A10)
- net SDA: now also R11.2, U1.18 (A4), TP1.1; no longer R11.1, U1.25 (A11)
- net T+: now reaches J1.1, U1.T+
- net at J1.2, J1.5: now also C9.2
- net T-: now reaches J1.3, U1.T-
- net R+: now reaches J1.4, U1.R+
- net R-: now reaches J1.6, U1.R-
- net nFAULT_1: now reaches U1.35 (TX8)
- net nFAULT_1: now also D1.1 (K), U2.35 (nFAULT), TP5.1
- removed net BSTA: C16.2, C25.1, C5.2, Q11.3 (S), Q12.1 (D), Q17.3 (S), Q18.1 (D), Q5.3 (S), Q6.1 (D), U2.10 (SHA), U4.10 (SHA), U5.10 (SHA)
- removed net BSTB: C17.2, C26.2, C6.2, Q1.3 (S), Q13.3 (S), Q14.1 (D), Q2.1 (D), Q7.3 (S), Q8.1 (D), U2.14 (SHB), U4.14 (SHB), U5.14 (SHB)
- removed net BSTC: C19.2, C27.2, C7.2, Q10.1 (D), Q15.3 (S), Q16.1 (D), Q3.3 (S), Q4.1 (D), Q9.3 (S), U2.18 (SHC), U4.18 (SHC), U5.18 (SHC)
- removed net CS: Q2.3 (S), Q6.3 (S), R16.2, R6.2, U2.21 (LSS), U2.22 (SP), U4.21 (LSS), U4.22 (SP)
- net GHA renamed GHA_1
- net GHA_1: no longer U4.11 (GHA), U5.11 (GHA)
- removed net GHB: R19.1, R24.1, R28.1, R34.1, R39.1, U2.15 (GLB), U4.15 (GLB), U5.15 (GLB)
- removed net GHC: R21.1, R26.1, R36.1, U2.19 (GHC), U4.19 (GHC), U5.19 (GHC)
- net GLA renamed GLA_1
- net GLA_1: no longer U4.12 (GLA), U5.12 (GLA)
- removed net GLB: R20.1, R25.1, R29.1, R35.1, R40.1, U2.15 (GLB), U4.15 (GLB), U5.15 (GLB)
- removed net GLC: R22.1, R27.1, R37.1, U2.20 (GLC), U4.20 (GLC), U5.20 (GLC)
- net PWM A (1) renamed PWM A_1
- net PWM A (2) renamed PWM A_2
- net PWM A (3) renamed PWM A_3
- net PWM B (1) renamed PWM B_1
- net PWM B (2) renamed PWM B_2
- net PWM B (3) renamed PWM B_3
- net PWM C (1) renamed PWM C_1
- net PWM C (2) renamed PWM C_2
- net PWM C (3) renamed PWM C_3
- net SCK: no longer names the net of U1.27 (A13)
- net SO (1) renamed SO_1
- net SO_1: now also TP4.1
- net SO (2) renamed SO_2
- net SO_2: now also TP10.1
- net SO (3) renamed SO_3
- net SO_3: now also TP16.1
- removed net nFAULT (1): D1.1 (K), U1.32 (OUT1B), U2.35 (nFAULT)
- net nFAULT (2) renamed nFAULT_2
- net nFAULT_2: now also TP11.1
- net nFAULT (3) renamed nFAULT_3
- net nFAULT_3: now also TP20.1
- net nSLEEP (1) renamed nSLEEP_1
- net nSLEEP (2) renamed nSLEEP_2
- net nSLEEP (3) renamed nSLEEP_3
- net nSLEEP_3: now also TP6.1
- new net: R33.1, U5.33 (CSAGAIN)
- new net: R1.2, U2.3 (DT)
- new net: R15.1, U4.33 (CSAGAIN)
- new net: R5.1, U2.33 (CSAGAIN)
- new net BSTA_1: C5.2, Conn2.1, Q5.3 (S), Q6.1 (D), TP13.1, U2.10 (SHA)
- new net BSTA_2: C16.2, Conn3.1, Q11.3 (S), Q12.1 (D), TP17.1, U4.10 (SHA)
- new net BSTA_3: C25.1, Conn4.1, Q17.3 (S), Q18.1 (D), TP24.1, U5.10 (SHA)
- new net BSTB_1: C6.2, Conn2.2, Q1.3 (S), Q2.1 (D), TP14.1, U2.14 (SHB)
- new net BSTB_2: C17.2, Conn3.2, Q7.3 (S), Q8.1 (D), TP18.1, U4.14 (SHB)
- new net BSTB_3: C26.2, Conn4.2, Q13.3 (S), Q14.1 (D), TP22.1, U5.14 (SHB)
- new net BSTC_1: C7.2, Conn2.3, Q3.3 (S), Q4.1 (D), TP15.1, U2.18 (SHC)
- new net BSTC_2: C19.2, Conn3.3, Q10.1 (D), Q9.3 (S), TP19.1, U4.18 (SHC)
- new net BSTC_3: C27.2, Conn4.3, Q15.3 (S), Q16.1 (D), TP23.1, U5.18 (SHC)
- new net GHA_2: R28.1, U4.11 (GHA)
- new net GHA_3: R39.1, U5.11 (GHA)
- new net GHB_1: R19.1, U2.15 (GHB)
- new net GHB_2: R24.1, U4.15 (GHB)
- new net GHB_3: R34.1, U5.15 (GHB)
- new net GHC_1: R21.1, U2.19 (GHC)
- new net GHC_2: R26.1, U4.19 (GHC)
- new net GHC_3: R36.1, U5.19 (GHC)
- new net GLA_2: R29.1, U4.12 (GLA)
- new net GLA_3: R40.1, U5.12 (GLA)
- new net GLB_1: R20.1, U2.16 (GLB)
- new net GLB_2: R25.1, U4.16 (GLB)
- new net GLB_3: R35.1, U5.16 (GLB)
- new net GLC_1: R22.1, U2.20 (GLC)
- new net GLC_2: R27.1, U4.20 (GLC)
- new net GLC_3: R37.1, U5.20 (GLC)
- no-connect marks 31 -> 32
Other:
- note added: "ACCELEROMETER CONNECTION"
- note added: "ETHERNET"
- note added: "GATE_DRIVER_1"
- note added: "GATE_DRIVER_2"
- note added: "GATE_DRIVER_3"
- note added: "MOSFETS_1"
- note added: "MOSFETS_2"
- note added: "MOSFETS_3"
- note added: "OKI"
- note added: "POWER ANDERSONS"
- note added: "POWER LEDS BULK CAPACITOR"
- note removed: "SI4156DY-T1-GE3"
- note removed: "deer"
- note removed: "then to MPU6050 breakout from Adafruit"
- moved on the sheet: C1, C10, C11, C12, C13, C14, C15, C16, C17, C19, C2, C20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

Commit message: Layout revisions
Layout revisions implemented from conversation with Drew
Edge cuts added
Vias added to ground planes
Ethernet connector moved to not attach to Teensey
Hopefully ready for order whenever next board order date is
Parts:
- J1: footprint Connector_RJ:RJ45_Connfly_DS1128-09-S8xx-S_Horizontal -> MRDT_Connectors:RJ45_Teensy
Changed lines of the file:
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@@
 			)
 		)
-		(property "Footprint" "Connector_RJ:RJ45_Connfly_DS1128-09-S8xx-S_Horizontal"
+		(property "Footprint" "MRDT_Connectors:RJ45_Teensy"
 			(at 226.06 32.385 90)
 			(effects

Commit message: Garrett Changes
Fixed some stray disconnected traces
Added mounting holes to schematic
Flipped ethernet port placement 180 degrees
Adjusted skew on Ethernet differential pairs
Replaced 470nf capacitor with correct 0603 ceramic capacitor (Was 470 uf and electrolytic)
Removed test points measurable directly from Teensey or Andersons
Parts:
- removed TP1, TP10, TP16, TP2, TP21, TP3, TP4, TP6, TP8, TP9: TestPoint, TestPoint:TestPoint_Pad_D2.0mm, symbol Connector:TestPoint
- added H1, H2, H3, H4: MountingHole, MountingHole:MountingHole_3mm, symbol Mechanical:MountingHole
- C15, C24: value 470 uF -> 470 nF; footprint Capacitor_THT:CP_Radial_D10.0mm_P5.00mm -> Capacitor_SMD:C_0603_1608Metric_Pad1.08x0.95mm_HandSolder
- C4: footprint Capacitor_THT:CP_Radial_D10.0mm_P5.00mm -> Capacitor_SMD:C_0603_1608Metric_Pad1.08x0.95mm_HandSolder
- U2, U4, U5: footprint DRV8329:VQFN40_RGF_TEX -> DRV8329:REE0036A-IPC_A
Connections:
- net BSTA_1 renamed SHA_1
- net BSTA_2 renamed SHA_2
- net BSTA_3 renamed SHA_3
- net BSTB_1 renamed SHB_1
- net BSTB_2 renamed SHB_2
- net BSTB_3 renamed SHB_3
- net BSTC_1 renamed SHC_1
- net BSTC_2 renamed SHC_2
- net BSTC_3 renamed SHC_3

Commit message: Final changes before ordering (hopefully)
Added a pin for the ground pad in the middle of the microcontrollers so it would actually connect to ground
Also added a via to the ground pad in the middle of the microcontroller because the schematic example had some
Put vias on some other non-connected ground plane areas
Connections:
- net GND: now also U2.37 (Ground), U4.37 (Ground), U5.37 (ground)
